Commit message: Fixed control law to see the measured wrench properly. Updated egm to display joint states with names, allowed us to view robot model in rviz. Changed params for stowage bay, and removed some debug output

File: irb120_description/urdf/irb120_w_ft_sensor.xacro (robot description, xacro)
@@ -15,7 +15,7 @@
   <xacro:include filename="$(find irb120_description)/urdf/materials.xacro" />
   <!-- Used for fixing robot to Gazebo 'base_link' -->
-  <link name="world"/>
+  <link name="map"/>
   <joint name="fixed" type="fixed">
-    <parent link="world"/>
+    <parent link="map"/>
     <child link="link1"/>
   </joint>
@@ -262,6 +262,6 @@
     <joint name="joint1">
       <hardwareInterface>PositionJointInterface</hardwareInterface>flange_stf
-[ INFO] [1512929221.358296873, 54.845000000]: frame_id: system_ref_frame
-[ INFO] [1512929221.358314256, 54.845000000]: child_frame_id: link7
+<!-- [ INFO] [1512929221.358296873, 54.845000000]: frame_id: system_ref_frame
+[ INFO] [1512929221.358314256, 54.845000000]: child_frame_id: link7 -->
     </joint>
     <actuator name="motor1">

Commit message: Updated RWE, Dithers, and added data collection node in current frame, small bug fixes

File: irb120_description/urdf/irb120_w_ft_sensor.xacro (robot description, xacro)
@@ -342,5 +342,5 @@
  		</inertial>
  	</link>
- 	<joint name = "ft_sensor_jnt" type = "continuous">
+ 	<joint name = "ft_sensor_jnt" type = "fixed">
  		<parent link = "link7"/>
  		<child link = "ft_sensor_link"/>

Commit message: Added gui pkg and updated state machines, minor bugfixs

File: irb120_description/urdf/irb120_w_ft_sensor.xacro (robot description, xacro)
@@ -84,5 +84,5 @@
 	<mesh filename="package://irb120_description/meshes/irb120/collision/link_1.stl"/>
       </geometry>
-      <material name="black"/>
+      <material name="orange"/>
     </visual>
     <inertial>
@@ -322,16 +322,16 @@
  	<link name = "ft_sensor_link">
  		<collision>
- 			<origin xyz ="0 0 0" rpy = "0 0 0"/>
+ 			<origin xyz ="0.04 0 0" rpy = "0 1.5708 0"/>
  			<geometry>
- 				<cylinder length = "0.001" radius = "0.001"/>
+ 				<cylinder length = "0.08" radius = "0.03"/>
  			</geometry>
  		</collision>
  		<visual>
- 			<origin xyz = "0 0 0" rpy = "0 0 0"/>
+ 			<origin xyz = "0.04 0 0" rpy = "0 1.5708 0"/>
  			<geometry>
- 				<cylinder length = "0.001" radius = "0.001"/>
+ 				<cylinder length = "0.08" radius = "0.03"/>
  			</geometry>
  			<material name = "ft_sensor_color">
- 				<color rgba = "1 0.5 0 1"/>
+ 				<color rgba = "0 0 0 1"/> <!-- was 1 0.5 0 1 -->
  			</material>
  		</visual>
